File: Kalid.kicad_pcb (KiCad board)
At the start: 2 copper layers, 116 parts, among them J1 USB_A, J2 USB-C Receptacle, J3 USB_A, J31 DC Connector, J4 USB_A, J5 USB_A, U1 TPS62933, U2 TPS62933, U3 GL3523-OTY30, U4 USB-PD, U5 LPW5209AB5F, U6 LPW5209AB5F, U7 LPW5209AB5F, U8 LPW5209AB5F, Y1 Crystal 25MHz 2016

Commit message: initial routing
Parts:
- added C40: Cap 4.7uF 0402, Capacitor_SMD:C_0402_1005Metric, F.Cu at (113.4, 81.2)
- added C41: Cap 22uF, Capacitor_SMD:C_0805_2012Metric, F.Cu at (186.0, 80.5)
- added C42: Cap 22uF, Capacitor_SMD:C_0805_2012Metric, F.Cu at (181.5, 80.5)
- added C43: Cap 4.7uF 0402, Capacitor_SMD:C_0402_1005Metric, F.Cu at (142.4, 83.1)
- added R44: R 0 ohm 0402, Resistor_SMD:R_0402_1005Metric, F.Cu at (103.8, 84.3)
- added R45: R 0 ohm 0402, Resistor_SMD:R_0402_1005Metric, F.Cu at (114.0, 83.0)
- added R46: R 5.1k 0402, Resistor_SMD:R_0402_1005Metric, F.Cu at (187.7, 69.2)
- added R47: R 5.1k 0402, Resistor_SMD:R_0402_1005Metric, F.Cu at (187.7, 71.1)
- added R48: R 5.1k 0402, Resistor_SMD:R_0402_1005Metric, F.Cu at (187.7, 72.1)
- added R49: R 5.1k 0402, Resistor_SMD:R_0402_1005Metric, F.Cu at (187.7, 68.2)
- added U9: W25Q128JVS, Package_SO:SOIC-8_5.3x5.3mm_P1.27mm, F.Cu at (108.9, 84.1)
- J1, J3, J4, J5: footprint Connector_USB:USB_A_Connfly_DS1095 -> Kalid:USB_A_Connfly_DS1095
- J2: footprint Connector_USB:USB_C_Receptacle_HRO_TYPE-C-31-M-12 -> Kalid:USB_C_Receptacle_HRO_TYPE-C-31-M-12
- moved D2 116.3 mm to (187.3, 101.8), turned to -90 degrees
- moved J1 114.6 mm to (175.1, 93.1)
- moved D3 99.8 mm to (169.9, 101.8), turned to -90 degrees
- moved R12 95.6 mm to (180.0, 82.2), turned to 90 degrees
- moved R13 95.6 mm to (180.0, 84.0), turned to -90 degrees
- moved D4 94.0 mm to (165.0, 101.8), turned to -90 degrees
- moved C32 93.7 mm to (185.7, 67.5), turned to 90 degrees
- moved C33 93.2 mm to (184.7, 67.5), turned to 90 degrees
- moved U5 92.6 mm to (172.2, 89.6), turned to 180 degrees
- moved J2 91.8 mm to (178.9, 68.7), turned to 180 degrees
- moved U4 90.5 mm to (186.0, 70.2), turned to -90 degrees
- moved R18 89.0 mm to (174.8, 88.5), turned to 90 degrees
- moved J3 87.8 mm to (152.8, 93.1)
- moved R43 87.1 mm to (183.8, 75.1)
- moved R42 86.7 mm to (183.4, 76.6)
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Connections:
- net Net-(J1-D+) renamed /Hierarchy/USB/P1_D+
- net Net-(J1-D-) renamed /Hierarchy/USB/P1_D-
- net Net-(J3-D+) renamed /Hierarchy/USB/P2_D+
- net Net-(J3-D-) renamed /Hierarchy/USB/P2_D-
- net Net-(J4-D+) renamed /Hierarchy/USB/P3_D+
- net Net-(J4-D-) renamed /Hierarchy/USB/P3_D-
- net Net-(J5-D+) renamed /Hierarchy/USB/P4_D+
- net Net-(J5-D-) renamed /Hierarchy/USB/P4_D-
- C21 pad 1: +V5V -> +1.2V
- R42 pad 1: unconnected-(R42-Pad1) -> Net-(U4-D-)
- R42 pad 2: /Hierarchy/USB/USB_UFP_D+ -> unconnected-(R42-Pad2)
- R43 pad 1: unconnected-(R43-Pad1) -> Net-(U4-D+)
- R43 pad 2: /Hierarchy/USB/USB_UFP_D- -> unconnected-(R43-Pad2)
- U3 pad 49: unconnected-(U3B-P_SPI_DO-Pad49) -> Net-(U3B-P_SPI_DO)
- U3 pad 50: unconnected-(U3B-P_SPI_CK-Pad50) -> Net-(U3B-P_SPI_CK)
- U3 pad 51: unconnected-(U3B-P_SPI_DI-Pad51) -> Net-(U3B-P_SPI_DI)
- U3 pad 52: unconnected-(U3B-P_SPI_CZ-Pad52) -> Net-(U3B-P_SPI_CZ)
Routing:
- net /Hierarchy/USB/P1_D+: track 0.00 -> 60.4 mm
- net /Hierarchy/USB/P1_D-: track 0.00 -> 60.4 mm
- net /Hierarchy/USB/USB_UFP_D+: track 0.00 -> 53.9 mm
- net /Hierarchy/USB/USB_UFP_D-: track 0.00 -> 53.9 mm
- net +V5V: track 0.00 -> 9.24 mm
Other:
- board outline added: 90 x 40 mm
- copper layers 2 -> 4

Commit message: finish routing
Parts:
- added C44: Cap 4.7uF 0402, Capacitor_SMD:C_0402_1005Metric, F.Cu at (147.8, 81.0)
- added H1: Mounting Hole, MountingHole:MountingHole_2.2mm_M2_DIN965_Pad_TopOnly, B.Cu at (122.5, 100.0)
- added H2: Mounting Hole, MountingHole:MountingHole_2.2mm_M2_DIN965_Pad_TopOnly, B.Cu at (165.0, 67.5)
- added H3: Mounting Hole, MountingHole:MountingHole_2.2mm_M2_DIN965_Pad_TopOnly, B.Cu at (117.5, 67.5)
- added H4: Mounting Hole, MountingHole:MountingHole_2.2mm_M2_DIN965_Pad_TopOnly, B.Cu at (167.5, 100.0)
- moved R14 13.0 mm to (146.6, 83.1), turned to -90 degrees
- moved R15 12.6 mm to (147.1, 82.6)
- moved R42 6.68 mm to (177.0, 74.9), turned to 180 degrees
- moved R41 4.73 mm to (178.0, 74.9), turned to 0 degrees
- moved R46 3.60 mm to (187.7, 72.8)
- moved R49 3.60 mm to (187.7, 71.8)
- moved R40 3.48 mm to (179.9, 77.0)
- moved R43 3.48 mm to (180.9, 77.0)
- moved R33 2.73 mm to (145.2, 98.7)
- moved R47 2.19 mm to (187.7, 68.9)
- moved R48 2.19 mm to (187.7, 69.9)
- moved C1 1.70 mm to (169.3, 68.8)
- moved C2 1.70 mm to (169.3, 66.8)
- moved C3 1.70 mm to (170.8, 74.8)
- moved C4 1.70 mm to (169.8, 74.8)
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Connections:
- net Net-(U1-SW) renamed /Hierarchy/Power/5VUSBSW
- net Net-(U2-SW) renamed /Hierarchy/Power/5VWALLSW
- C32 pad 1: +V5V -> +VUSBIN
- U4 pad 2: +V5V -> +VUSBIN
Routing:
- net GND: track 0.00 -> 136.6 mm, vias 0 -> 156
- net +V5VWALL: track 0.00 -> 97.6 mm, vias 0 -> 11
- net Net-(U3B-RESETJ): track 0.00 -> 83.4 mm, vias 0 -> 2
- net +3.3V: track 0.00 -> 77.4 mm, vias 0 -> 11
- net Net-(D2-A): track 0.00 -> 69.7 mm, vias 0 -> 2
- net Net-(D9-A): track 0.00 -> 67.6 mm, vias 0 -> 2
- net Net-(U3B-P_SPI_DO): track 0.00 -> 67.1 mm, vias 0 -> 2
- net Net-(U3B-P_SPI_DI): track 0.00 -> 60.6 mm, vias 0 -> 2
- net Net-(U3B-P_SPI_CK): track 0.00 -> 60.1 mm, vias 0 -> 2
- net Net-(D3-A): track 0.00 -> 59.9 mm, vias 0 -> 2
- net Net-(D8-A): track 0.00 -> 58.0 mm, vias 0 -> 2
- net Net-(U3G-OVCUR4J/SMD): track 0.00 -> 48.9 mm, vias 0 -> 2
- net Net-(U3B-P_SPI_CZ): track 0.00 -> 48.5 mm, vias 0 -> 2
- net /Hierarchy/USB/P4_D-: track 0.00 -> 47.8 mm
- net /Hierarchy/USB/P4_D+: track 0.00 -> 47.4 mm
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- added copper zone on In2.Cu, net +1.2V
- added copper zone on B.Cu, net +3.3V
- added copper zone on In2.Cu, net +V5V
- added copper zone on F.Cu, net +V5VUSB
- added copper zone on In2.Cu, net +V5VUSB
- added copper zone on F.Cu, net +V5VWALL
- added copper zone on In2.Cu, net +V5VWALL
- added copper zone on F.Cu, net /Hierarchy/Power/5VUSBSW
- added copper zone on F.Cu, net /Hierarchy/Power/5VWALLSW
- added copper zone on B.Cu, net GND
- added copper zone on F.Cu, net GND
- added copper zone on In1.Cu, net GND
Other:
- outline, holes or cut-outs redrawn
- board text added: "(Optional)"
- board text added: "5-20V"
- board text added: "5V"
- board text added: "5VUSB"
- board text added: "5VWALL"
- board text added: "EVT1 27/7/2026"
- board text added: "Kalid"
- board text added: "OVCUR"
- board text added: "PORT 1"
- board text added: "PORT 2"
- board text added: "PORT 3"
- board text added: "PORT 4"
- board text added: "Switchable USB Hub"
