File: Kalid.kicad_pcb (KiCad board)
At the start: 4 copper layers, 90 x 40 mm, 148 parts, among them J1 USB_A, J2 USB_C_Receptacle, J3 USB_A, J31 DC Connector, J4 USB_A, J5 USB_A, J6 Conn_01x04, U1 TPS62933, U2 TPS62933, U3 GL3523-OTY30, U4 USB-PD, U5 LPW5209AB5F, U6 LPW5209AB5F, U7 LPW5209AB5F, U8 LPW5209AB5F, U9 W25Q128JVS, Y1 Crystal 25MHz 2016

Commit message: release evt5
Parts:
- removed J2: USB_C_Receptacle, Kalid:USB-C-SMD_TYPE-C-24P-QT
- removed R47, R48, R49: R 5.1k 0402, Resistor_SMD:R_0402_1005Metric
- added C44: Cap 22uF, Capacitor_SMD:C_0805_2012Metric, F.Cu at (156.9, 82.6)
- added C45: Cap 22uF, Capacitor_SMD:C_0805_2012Metric, F.Cu at (158.9, 84.2)
- added C46: Cap 22uF, Capacitor_SMD:C_0805_2012Metric, F.Cu at (115.5, 83.7)
- added C47: Cap 22uF, Capacitor_SMD:C_0805_2012Metric, F.Cu at (117.5, 83.7)
- added J7: USB_C_Receptacle_USB2.0_16P, Kalid:USB_C_Receptacle_HRO_TYPE-C-31-M-12, F.Cu at (179.1, 69.0)
- added R40: R 1M 0402, Resistor_SMD:R_0402_1005Metric, F.Cu at (151.8, 72.9)
- added R41: R 0 ohm 0402, Resistor_SMD:R_0402_1005Metric, F.Cu at (102.8, 82.2)
- added R42: R 0 ohm 0402, Resistor_SMD:R_0402_1005Metric, F.Cu at (102.8, 83.2)
- added R43: R 0 ohm 0402, Resistor_SMD:R_0402_1005Metric, F.Cu at (103.2, 82.7)
- R46: value R 5.1k 0402 -> R 0 ohm 0402
- U9: value W25Q128JVS -> MX25L1006EMI-10G
- moved R46 86.0 mm to (102.3, 82.7), turned to -90 degrees
- moved TP8 3.20 mm to (101.7, 79.5)
- moved C27 0.57 mm to (140.7, 71.2)
- moved TP7 0.50 mm to (185.5, 75.0)
- moved C32 0.36 mm to (186.1, 67.6)
- moved C33 0.36 mm to (185.1, 67.6)
- moved U4 0.36 mm to (186.3, 70.3)
- moved D6 0.11 mm to (125.2, 101.9)
- moved R26 0.11 mm to (125.2, 99.7)
- moved R22 0.05 mm to (154.6, 83.0)
Connections:
- R46 pad 1: GND -> /Hierarchy/USB/SPI_COPI
- R46 pad 2: /Hierarchy/USB/CC2 -> Net-(U3B-P_SPI_DI)
- U3 pad 49: /Hierarchy/USB/SPI_CIPO -> Net-(U3B-P_SPI_DO)
- U3 pad 51: /Hierarchy/USB/SPI_COPI -> Net-(U3B-P_SPI_DI)
- U3 pad 68: /Hierarchy/USB/USB_UFP_TX- -> unconnected-(U3C-TXN1_P0-Pad68)
- U3 pad 69: /Hierarchy/USB/USB_UFP_TX+ -> unconnected-(U3C-TXP1_P0-Pad69)
- U3 pad 71: /Hierarchy/USB/USB_UFP_RX- -> unconnected-(U3C-RXN1_P0-Pad71)
- U3 pad 72: /Hierarchy/USB/USB_UFP_RX+ -> unconnected-(U3C-RXP1_P0-Pad72)
Routing:
- net Net-(U3B-P_SPI_DO): track 0.00 -> 67.1 mm, vias 0 -> 2
- net Net-(U3B-P_SPI_DI): track 0.00 -> 66.7 mm, vias 0 -> 3
- net /Hierarchy/USB/USB_UFP_RX+: track 64.1 -> 0.00 mm, vias 2 -> 0
- net /Hierarchy/USB/USB_UFP_RX-: track 64.1 -> 0.00 mm, vias 2 -> 0
- net /Hierarchy/USB/SPI_CIPO: track 64.8 -> 2.31 mm, vias 2 -> 0
- net /Hierarchy/USB/USB_UFP_TX+: track 60.5 -> 0.00 mm, vias 2 -> 0
- net /Hierarchy/USB/USB_UFP_TX-: track 60.5 -> 0.00 mm, vias 2 -> 0
- net /Hierarchy/USB/SPI_COPI: track 59.3 -> 13.5 mm, vias 2 -> 0
- net +3.3V: track 138.1 -> 154.8 mm, vias 12 -> 13
- net /Hierarchy/USB/P4_D-: track 47.1 -> 38.3 mm
- net /Hierarchy/USB/P4_D+: track 47.1 -> 38.3 mm
- net +1.2V: track 76.6 -> 85.2 mm, vias 7 -> 8
- net +VUSBIN: track 49.4 -> 42.2 mm, vias 11 -> 10
- net GND: track 145.4 -> 141.8 mm, vias 168 -> 162
- net /Hierarchy/USB/USB_UFP_D-: track 64.9 -> 62.3 mm
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Other:
- board text added: "EVT5 18/9/2026"
- board text added: "Manufacture with JLC04161H-7628(Standard/Finished thickness1.59mm±10%) 90 ohm impedance has trace width of 1397, trace spacing of 0.1016mm, and impedance trace-to-copper of 0.1016mm"
- board text removed: "EVT4 4/9/2026"
- board text removed: "Manufacture with JLC04161H-7628(Standard/Finished thickness1.59mm±10%) 90 ohm impedance has trace spacing of 0.12mm and impedance trace-to-copper of 0.2mm"
