File: Hierarchy.kicad_sch (KiCad schematic)
At the start: 0 parts

Commit message: tag schematic and pcb as evt2
Other:
- title: (none) -> Kalid
Changed lines of the file:
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@@
 	(generator_version "9.0")
 	(paper "A4")
+	(title_block
+		(title "Kalid")
+		(date "2025-08-18")
+		(rev "EVT2")
+	)
 	(sheet
 		(at 62.23 80.01)
